Commit message: fixing stuff

File: description/robot_core.xacro (robot description, xacro)
@@ -41,4 +41,5 @@
         </visual>
     </link>
+    <!-- Need to fix xyz to match other joints-->
     <joint name="wheel_arm_LF_joint" type="fixed" >
         <parent link="chassis_link"/>
@@ -97,5 +98,5 @@
         <parent link="wheel_arm_LF_link"/>
         <child link="wheel_LF_link" type="fixed"/>
-        <origin rpy="0 0 0" xyz="-.038 0 0" />
+        <origin rpy="0 0 0" xyz="0 -.125 0" />
     </joint>
     <link name="wheel_LF_link">
@@ -107,3 +108,29 @@
         </visual>
     </link>
+    <joint name="wheel_RR_joint" type="fixed">
+        <parent link="wheel_arm_RR_link"/>
+        <child link="wheel_RR_link" type="fixed"/>
+        <origin rpy="0 -1.5708 0" xyz="0 -.125 -.038" />
+    </joint>
+    <link name="wheel_RR_link">
+        <visual>
+        <origin rpy="0 0 0" xyz="0 0 0"/>
+        <geometry>
+            <mesh filename="file:///home/joel/dev_ws/src/rover_one/description/G_Wheel.dae" scale="1 1 1"/>
+        </geometry>
+        </visual>
+    </link>
+    <joint name="wheel_LR_joint" type="fixed">
+        <parent link="wheel_arm_LR_link"/>
+        <child link="wheel_LR_link" type="fixed"/>
+        <origin rpy="0 0 0" xyz="0 -.125 0" />
+    </joint>
+    <link name="wheel_LR_link">
+        <visual>
+        <origin rpy="0 0 0" xyz="0 0 0"/>
+        <geometry>
+            <mesh filename="file:///home/joel/dev_ws/src/rover_one/description/G_Wheel.dae" scale="1 1 1"/>
+        </geometry>
+        </visual>
+    </link>
 </robot>

Commit message: Fixing joints and adding collisions

File: description/robot_core.xacro (robot description, xacro)
@@ -1,16 +1,4 @@
 <?xml version="1.0"?>
 <robot xmlns:xacro="http://www.ros.org/wiki/xacro" >
-    <material name="white">
-        <color rgba="1 1 1 1" />
-    </material>
-    <material name="orange">
-        <color rgba="1 0.3 0.1 1" />
-    </material>
-    <material name="blue">
-        <color rgba="0.2 0.2 1 1" />
-    </material>
-    <material name="black">
-        <color rgba="0 0 0 1" />
-    </material>
     <link name="base_link">
     </link>
@@ -22,115 +10,181 @@
     <link name="chassis_link">
         <visual>
-            <origin rpy="1.5708 0 0" xyz="0 0 .01" />
+            <origin rpy="${pi/2} 0 0" xyz="0 0 .01" />
             <geometry>
                 <mesh filename="file:///home/joel/dev_ws/src/rover_one/description/G_Assy_Base.dae" scale="1 1 1"/>
             </geometry>
         </visual>
+        <collision>
+            <origin rpy="${pi/2} 0 0" xyz="0 0 .01" />
+            <geometry>
+                <mesh filename="file:///home/joel/dev_ws/src/rover_one/description/G_Assy_Base.dae" scale="1 1 1"/>
+            </geometry>
+        </collision>
     </link>
-    <joint name="wheel_arm_RF_joint" type="fixed" >
+    <joint name="wheel_arm_RF_joint" type="revolute" >
         <parent link="chassis_link"/>
         <child link="wheel_arm_RF_link" />
         <origin rpy="0 0 0" xyz="-.2 -.15 .0375" />
+        <axis xyz="0 0 1"/>
+        <limit lower="0.7854" upper="-0.7854" effort="10.0" velocity="2.0"/>
     </joint>
     <link name="wheel_arm_RF_link" >
         <visual>
-        <origin rpy="1.5708 0 1.5708" xyz="0 0 0"/>+
-        <geometry>
-            <mesh filename="file:///home/joel/dev_ws/src/rover_one/description/G_Wheel_Arm.dae" scale="1 1 1"/>
-        </geometry>
+            <origin rpy="${pi/2} 0 ${pi/2}" xyz="0 0 0"/>+
+            <geometry>
+                <mesh filename="file:///home/joel/dev_ws/src/rover_one/description/G_Wheel_Arm.dae" scale="1 1 1"/>
+            </geometry>
         </visual>
+        <collision>
+            <origin rpy="${pi/2} 0 ${pi/2}" xyz="0 0 0"/>+
+            <geometry>
+                <mesh filename="file:///home/joel/dev_ws/src/rover_one/description/G_Wheel_Arm.dae" scale="1 1 1"/>
+            </geometry>
+        </collision>
     </link>
-    <!-- Need to fix xyz to match other joints-->
-    <joint name="wheel_arm_LF_joint" type="fixed" >
+    <joint name="wheel_arm_LF_joint" type="revolute" >
         <parent link="chassis_link"/>
         <child link="wheel_arm_LF_link" />
-        <origin rpy="1.5708 0 -1.5708" xyz=".2 -.15 .0375" />
+        <origin rpy="0 0 0" xyz=".2 -.15 .0375" />
+        <axis xyz="0 0 1"/>
+        <limit lower="0.7854" upper="-0.7854" effort="10.0" velocity="2.0"/>
     </joint>
     <link name="wheel_arm_LF_link" >
         <visual>
-        <origin rpy="0 0 0" xyz="0 0 0"/>+
-        <geometry>
-            <mesh filename="file:///home/joel/dev_ws/src/rover_one/description/G_Wheel_Arm.dae" scale="1 1 1"/>
-        </geometry>
+            <origin rpy="${pi/2} 0 -${pi/2}" xyz="0 0 0"/>+
+            <geometry>
+                <mesh filename="file:///home/joel/dev_ws/src/rover_one/description/G_Wheel_Arm.dae" scale="1 1 1"/>
+            </geometry>
         </visual>
+        <collision>
+            <origin rpy="${pi/2} 0 -${pi/2}" xyz="0 0 0"/>+
+            <geometry>
+                <mesh filename="file:///home/joel/dev_ws/src/rover_one/description/G_Wheel_Arm.dae" scale="1 1 1"/>
+            </geometry>
+        </collision>
     </link>
-    <!--Red x, blue y, green z -->
-    <joint name="wheel_arm_RR_joint" type="fixed" >
+    <!--Red x, green y, blue z -->
+    <joint name="wheel_arm_RR_joint" type="revolute" >
         <parent link="chassis_link"/>
         <child link="wheel_arm_RR_link" />
-        <origin rpy="1.5708 0 1.5708" xyz="-.2 .15 .0375" />
+        <origin rpy="0 0 0" xyz="-.2 .15 .0375" />
+        <axis xyz="0 0 1"/>
+        <limit lower="0.7854" upper="-0.7854" effort="10.0" velocity="2.0"/>
     </joint>
     <link name="wheel_arm_RR_link" >
         <visual>
-        <origin rpy="0 0 0" xyz="0 0 0"/>+
-        <geometry>
-            <mesh filename="file:///home/joel/dev_ws/src/rover_one/description/G_Wheel_Arm.dae" scale="1 1 1"/>
-        </geometry>
+            <origin rpy="${pi/2} 0 ${pi/2}" xyz="0 0 0"/>+
+            <geometry>
+                <mesh filename="file:///home/joel/dev_ws/src/rover_one/description/G_Wheel_Arm.dae" scale="1 1 1"/>
+            </geometry>
         </visual>
+        <collision>
+            <origin rpy="${pi/2} 0 ${pi/2}" xyz="0 0 0"/>+
+            <geometry>
+                <mesh filename="file:///home/joel/dev_ws/src/rover_one/description/G_Wheel_Arm.dae" scale="1 1 1"/>
+            </geometry>
+        </collision>
     </link>
-    <joint name="wheel_arm_LR_joint" type="fixed" >
+    <joint name="wheel_arm_LR_joint" type="revolute" >
         <parent link="chassis_link"/>
         <child link="wheel_arm_LR_link" />
-        <origin rpy="1.5708 0 -1.5708" xyz=".2 .15 .0375" />
+        <origin rpy="0 0 0" xyz=".2 .15 .0375" />
+        <axis xyz="0 0 1"/>
+        <limit lower="0.7854" upper="-0.7854" effort="10.0" velocity="2.0"/>
     </joint>
     <link name="wheel_arm_LR_link" >
         <visual>
-        <origin rpy="0 0 0" xyz="0 0 0"/>
-        <geometry>
-            <mesh filename="file:///home/joel/dev_ws/src/rover_one/description/G_Wheel_Arm.dae" scale="1 1 1"/>
-        </geometry>
+            <origin rpy="${pi/2} 0 -${pi/2}" xyz="0 0 0"/>
+            <geometry>
+                <mesh filename="file:///home/joel/dev_ws/src/rover_one/description/G_Wheel_Arm.dae" scale="1 1 1"/>
+            </geometry>
         </visual>
+        <collision>
+            <origin rpy="${pi/2} 0 -${pi/2}" xyz="0 0 0"/>
+            <geometry>
+                <mesh filename="file:///home/joel/dev_ws/src/rover_one/description/G_Wheel_Arm.dae" scale="1 1 1"/>
+            </geometry>
+        </collision>
     </link>
-    <joint name="wheel_RF_joint" type="fixed">
+    <!-- Wheels -->
+    <joint name="wheel_RF_joint" type="continuous">
         <parent link="wheel_arm_RF_link"/>
-        <child link="wheel_RF_link" type="fixed"/>
+        <child link="wheel_RF_link" />
         <origin rpy="0 0 0" xyz="-.038 0 -.125" />
+        <axis xyz="1 0 0"/>
     </joint>
     <link name="wheel_RF_link">
         <visual>
-        <origin rpy="0 0 0" xyz="0 0 0"/>
-        <geometry>
-            <mesh filename="file:///home/joel/dev_ws/src/rover_one/description/G_Wheel.dae" scale="1 1 1"/>
-        </geometry>
+            <origin rpy="0 0 0" xyz="0 0 0"/>
+            <geometry>
+                <mesh filename="file:///home/joel/dev_ws/src/rover_one/description/G_Wheel.dae" scale="1 1 1"/>
+            </geometry>
         </visual>
+        <collision>
+            <origin rpy="0 0 0" xyz="0 0 0"/>
+            <geometry>
+                <mesh filename="file:///home/joel/dev_ws/src/rover_one/description/G_Wheel.dae" scale="1 1 1"/>
+            </geometry>
+        </collision>
     </link>
-    <joint name="wheel_LF_joint" type="fixed">
+    <joint name="wheel_LF_joint" type="continuous">
         <parent link="wheel_arm_LF_link"/>
-        <child link="wheel_LF_link" type="fixed"/>
-        <origin rpy="0 0 0" xyz="0 -.125 0" />
+        <child link="wheel_LF_link" />
+        <origin rpy="0 0 0" xyz=".038 0 -.125" />
+        <axis xyz="1 0 0"/>
     </joint>
     <link name="wheel_LF_link">
         <visual>
-        <origin rpy="0 0 0" xyz="0 0 0"/>
-        <geometry>
-            <mesh filename="file:///home/joel/dev_ws/src/rover_one/description/G_Wheel.dae" scale="1 1 1"/>
-        </geometry>
+            <origin rpy="0 0 ${pi}" xyz="0 0 0"/>
+            <geometry>
+                <mesh filename="file:///home/joel/dev_ws/src/rover_one/description/G_Wheel.dae" scale="1 1 1"/>
+            </geometry>
         </visual>
+        <collision>
+            <origin rpy="0 0 ${pi}" xyz="0 0 0"/>
+            <geometry>
+                <mesh filename="file:///home/joel/dev_ws/src/rover_one/description/G_Wheel.dae" scale="1 1 1"/>
+            </geometry>
+        </collision>
     </link>
-    <joint name="wheel_RR_joint" type="fixed">
+    <joint name="wheel_RR_joint" type="continuous">
         <parent link="wheel_arm_RR_link"/>
-        <child link="wheel_RR_link" type="fixed"/>
-        <origin rpy="0 -1.5708 0" xyz="0 -.125 -.038" />
+        <child link="wheel_RR_link"/>
+        <origin rpy="0 0 0" xyz="-.038 0 -.125" />
+        <axis xyz="1 0 0"/>
     </joint>
     <link name="wheel_RR_link">
         <visual>
-        <origin rpy="0 0 0" xyz="0 0 0"/>
-        <geometry>
-            <mesh filename="file:///home/joel/dev_ws/src/rover_one/description/G_Wheel.dae" scale="1 1 1"/>
-        </geometry>
+            <origin rpy="0 0 0" xyz="0 0 0"/>
+            <geometry>
+                <mesh filename="file:///home/joel/dev_ws/src/rover_one/description/G_Wheel.dae" scale="1 1 1"/>
+            </geometry>
         </visual>
+        <collision>
+            <origin rpy="0 0 0" xyz="0 0 0"/>
+            <geometry>
+                <mesh filename="file:///home/joel/dev_ws/src/rover_one/description/G_Wheel.dae" scale="1 1 1"/>
+            </geometry>
+        </collision>
     </link>
-    <joint name="wheel_LR_joint" type="fixed">
+    <joint name="wheel_LR_joint" type="continuous">
         <parent link="wheel_arm_LR_link"/>
-        <child link="wheel_LR_link" type="fixed"/>
-        <origin rpy="0 0 0" xyz="0 -.125 0" />
+        <child link="wheel_LR_link" />
+        <origin rpy="0 0 0" xyz=".038 0 -.125" />
+        <axis xyz="1 0 0"/>
     </joint>
     <link name="wheel_LR_link">
         <visual>
-        <origin rpy="0 0 0" xyz="0 0 0"/>
-        <geometry>
-            <mesh filename="file:///home/joel/dev_ws/src/rover_one/description/G_Wheel.dae" scale="1 1 1"/>
-        </geometry>
+            <origin rpy="0 0 ${pi}" xyz="0 0 0"/>
+            <geometry>
+                <mesh filename="file:///home/joel/dev_ws/src/rover_one/description/G_Wheel.dae" scale="1 1 1"/>
+            </geometry>
         </visual>
+        <collision>
+        <origin rpy="0 0 ${pi}" xyz="0 0 0"/>
+            <geometry>
+                <mesh filename="file:///home/joel/dev_ws/src/rover_one/description/G_Wheel.dae" scale="1 1 1"/>
+            </geometry>
+        </collision>
     </link>
 </robot>

Commit message: adding stuff

File: description/robot_core.xacro (robot description, xacro)
@@ -1,4 +1,6 @@
 <?xml version="1.0"?>
 <robot xmlns:xacro="http://www.ros.org/wiki/xacro" >
+    <xacro:include filename="inertial_macros.xacro"/>
+    <!-- add this to links-->
     <link name="base_link">
     </link>
@@ -21,4 +23,7 @@
             </geometry>
         </collision>
+        <xacro:inertial_box mass="0.5" x="0.3" y="0.3" z="0.15">
+            <origin xyz="0 0 .01" rpy="0 0 0"/>
+        </xacro:inertial_box>
     </link>
     <joint name="wheel_arm_RF_joint" type="revolute" >

Commit message: fixing more stuff, im new!

File: description/robot_core.xacro (robot description, xacro)
@@ -1,6 +1,4 @@
 <?xml version="1.0"?>
 <robot xmlns:xacro="http://www.ros.org/wiki/xacro" >
-    <xacro:include filename="inertial_macros.xacro"/>
-    <!-- add this to links-->
     <link name="base_link">
     </link>
@@ -23,7 +21,4 @@
             </geometry>
         </collision>
-        <xacro:inertial_box mass="0.5" x="0.3" y="0.3" z="0.15">
-            <origin xyz="0 0 .01" rpy="0 0 0"/>
-        </xacro:inertial_box>
     </link>
     <joint name="wheel_arm_RF_joint" type="revolute" >
@@ -181,7 +176,7 @@
     <link name="wheel_LR_link">
         <visual>
-            <origin rpy="0 0 ${pi}" xyz="0 0 0"/>
-            <geometry>
-                <mesh filename="file:///home/joel/dev_ws/src/rover_one/description/G_Wheel.dae" scale="1 1 1"/>
+        <origin rpy="0 0 ${pi}" xyz="0 0 0"/>
+        <geometry>
+            <mesh filename="file:///home/joel/dev_ws/src/rover_one/description/G_Wheel.dae" scale="1 1 1"/>
             </geometry>
         </visual>
